File: PCBs/supervision/RTU.brd (EAGLE design)
At the start: 75 x 59 mm, 17 parts, among them IC1 LM1117T-1.8, IC2 7805T, M1 WIRELESS-NRF24L01, U1 ESP-WROOM-32, U2 MICROSD_CATALEX, U3 DS1307Z, Y2 32kHz

Commit message: Alterações na PCB do sistema supervisorio
Parts:
- added Q1: BC548, transistor-npn:TO92-EBC
Connections:
- new net GND_SD: Q1.C, U2.GND
- net CS: now also Q1.B
- net GND: now also Q1.E; no longer U2.GND
Routing:
- net CS: track 43.2 -> 71.2 mm
- net GND_SD: track 0.00 -> 7.87 mm
- net 5V: track 67.4 -> 64.4 mm
Changed lines of the file:
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@@
 <drawing>
 <settings>
-<setting alwaysvectorfont="no"/>
+<setting alwaysvectorfont="yes"/>
 <setting verticaltext="up"/>
 </settings>
@@
 </layers>
 <board>
+<fusionsync huburn="a.cGVyc29uYWw6dWUyY2NiZmI4" projecturn="a.cGVyc29uYWw6dWUyY2NiZmI4IzIwMTkwMTI0MTcyMjcyMTUx" f3durn="urn:adsk.wipprod:dm.lineage:vljMM_kDTuCh9VKP5X2PJw" pcbguid="a6e1b2c5-2a28-44fb-b83e-43568e824d7c" lastpulledtime="" lastsyncedchangeguid="cf847ee6-e7db-db41-a710-733bcf0a3aec"/>
 <plain>
 <wire x1="0" y1="59" x2="0" y2="0" width="0" layer="20"/>
@@
 <attribute name="VALUE" x="51.215" y="41.092" size="1.27" layer="27" ratio="10" rot="R90"/>
 </element>
+<element name="Q1" library="transistor-npn" library_urn="urn:adsk.eagle:library:398" package="TO92-EBC" package3d_urn="urn:adsk.eagle:package:28989/2" value="BC548" x="29.6" y="56.7" smashed="yes">
+<attribute name="NAME" x="27.06" y="58.478" size="1.27" layer="25" ratio="10"/>
+<attribute name="VALUE" x="27.06" y="52.128" size="1.27" layer="27" ratio="10"/>
+</element>
 </elements>
 <signals>
@@
 <contactref element="RESET_BUTTON" pad="1"/>
 <contactref element="M1" pad="1"/>
-<contactref element="U2" pad="GND"/>
 <contactref element="C3" pad="2"/>
 <contactref element="C4" pad="2"/>
@@
 <contactref element="U3" pad="4"/>
 <contactref element="G2" pad="-"/>
+<contactref element="Q1" pad="E"/>
+<wire x1="16.37" y1="23.04" x2="7.42" y2="30.74" width="0" layer="19" extent="16-16"/>
 </signal>
 <signal name="3.3V">
@@
 <wire x1="9.7" y1="42.1" x2="9.7" y2="49.73" width="0.508" layer="16"/>
 <wire x1="9.7" y1="49.73" x2="9.75" y2="49.78" width="0.508" layer="16"/>
+<wire x1="9.75" y1="49.78" x2="9.75" y2="55.05" width="0.8128" layer="16"/>
+<wire x1="12.2776" y1="57.5776" x2="29" y2="57.5776" width="0.8128" layer="16"/>
+<wire x1="9.75" y1="55.05" x2="12.2776" y2="57.5776" width="0.8128" layer="16"/>
+<contactref element="Q1" pad="B"/>
+<wire x1="29" y1="57.5776" x2="29.6" y2="56.9776" width="0.8128" layer="16"/>
+<wire x1="29.6" y1="56.9776" x2="29.6" y2="55.43" width="0.8128" layer="16"/>
 </signal>
 <signal name="N$1">
@@
 <contactref element="U2" pad="VCC"/>
 <wire x1="34.18" y1="45.01" x2="30.89" y2="45.01" width="0.8128" layer="16"/>
-<wire x1="29" y1="46.9" x2="29" y2="49.9" width="0.8128" layer="16"/>
-<wire x1="29" y1="49.9" x2="26.5" y2="52.4" width="0.8128" layer="16"/>
-<wire x1="26.5" y1="52.4" x2="21" y2="52.4" width="0.8128" layer="16"/>
-<wire x1="21" y1="52.4" x2="19.91" y2="51.31" width="0.8128" layer="16"/>
-<wire x1="19.91" y1="51.31" x2="19.91" y2="49.78" width="0.8128" layer="16"/>
-<wire x1="30.89" y1="45.01" x2="29" y2="46.9" width="0.8128" layer="16"/>
 <wire x1="40.34" y1="47.18" x2="40.34" y2="39.36" width="0.508" layer="16"/>
 <wire x1="40.34" y1="39.36" x2="43" y2="36.7" width="0.508" layer="16"/>
 <wire x1="43" y1="36.7" x2="43.035" y2="36.735" width="0.508" layer="16"/>
 <wire x1="43.035" y1="36.735" x2="45.91" y2="36.735" width="0.508" layer="16"/>
+<wire x1="30.89" y1="45.01" x2="21.59" y2="45.01" width="0.8128" layer="16"/>
+<wire x1="21.59" y1="45.01" x2="19.9" y2="46.7" width="0.8128" layer="16"/>
+<wire x1="19.9" y1="46.7" x2="19.9" y2="49.77" width="0.8128" layer="16"/>
+<wire x1="19.9" y1="49.77" x2="19.91" y2="49.78" width="0.8128" layer="16"/>
 </signal>
 <signal name="SCL">
@@
 <wire x1="10.2" y1="25.3" x2="9.29" y2="24.39" width="0.508" layer="16"/>
 </signal>
+<signal name="GND_SD">
+<contactref element="Q1" pad="C"/>
+<contactref element="U2" pad="GND"/>
+<wire x1="22.45" y1="49.78" x2="22.45" y2="51.35" width="0.8128" layer="16"/>
+<wire x1="26.53" y1="55.43" x2="27.06" y2="55.43" width="0.8128" layer="16"/>
+<wire x1="22.45" y1="51.35" x2="26.53" y2="55.43" width="0.8128" layer="16"/>
+</signal>
 </signals>
 <mfgpreviewcolors>
@@
 </note>
 <note version="8.3" severity="warning">
+Since Version 8.3, EAGLE supports Fusion synchronisation.
+This feature will not be available in this version and saving
+the document will break the link to the Fusion PCB feature.
+</note>
+<note version="8.3" severity="warning">
